Commit message: adding gripper to kuka ee

File: src/kuka_robot_descriptions/kuka_cybertech_support/urdf/kr16_r2010_2.urdf.xacro (robot description, xacro)
@@ -4,4 +4,5 @@
   <xacro:include filename="$(find kuka_cybertech_support)/urdf/kr16_r2010_2_macro.xacro"/>
   <xacro:include filename="$(find kuka_cybertech_support)/urdf/kr_cybertech_ros2_control_macro.xacro"/>
+  <xacro:include filename="$(find gripper_ee_description)/urdf/gripper_ee_macro.xacro"/>
   <!-- Read additional arguments  -->
   <xacro:arg name="driver_version" default="eki_rsi"/>
@@ -34,3 +35,7 @@
     <origin xyz="$(arg x) $(arg y) $(arg z)" rpy="$(arg roll) $(arg pitch) $(arg yaw)"/>
   </joint>
+  <!-- gripper end effector mounted on the robot flange -->
+  <xacro:gripper_ee prefix="$(arg prefix)" parent="$(arg prefix)flange">
+    <origin xyz="0 0 0" rpy="0 0 0"/>
+  </xacro:gripper_ee>
 </robot>
