Commit message: updated kuka setup

File: src/kuka_robot_descriptions/kuka_cybertech_support/urdf/kr16_r2010_2.urdf (robot description, URDF)
Before this commit: robot kr16_r2010_2, 11 links, 10 joints
Links:
- link base_link: mass None -> 6.5E1
- link link_1: mass None -> 8.4207E1
- link link_2: mass None -> 5.5E1
- link link_3: mass None -> 1.5E1
- link link_4: mass None -> 1.2E1
- link link_5: mass None -> 5.0
- link link_6: mass None -> 4.0

File: src/kuka_robot_descriptions/kuka_cybertech_support/urdf/kr16_r2010_2_macro.xacro (robot description, xacro)
@@ -10,4 +10,9 @@
         <origin rpy="-0.0 0.0 -0.0" xyz="0.0 0.0 0.0"/>
       </collision>
+      <inertial>
+        <mass value="6.5E1"/>
+        <origin rpy="0.0 0.0 0.0" xyz="0.0 0.0 0.15"/>
+        <inertia ixx="1.0" ixy="0.0" ixz="0.0" iyy="1.0" iyz="0.0" izz="1.5"/>
+      </inertial>
       <visual>
         <geometry>
@@ -15,4 +20,7 @@
         </geometry>
         <origin rpy="-0.0 0.0 -0.0" xyz="0.0 0.0 0.0"/>
+        <material name="KukaOrange">
+          <color rgba="1.0 0.4 0.0 1.0"/>
+        </material>
       </visual>
     </link>
@@ -24,4 +32,9 @@
         <origin rpy="-0.0 0.0 -0.0" xyz="0.0 0.0 0.0"/>
       </collision>
+      <inertial>
+        <mass value="8.4207E1"/>
+        <origin rpy="0.0 0.0 0.0" xyz="0.05 0.005 -0.26"/>
+        <inertia ixx="2.0" ixy="0.0" ixz="0.0" iyy="2.0" iyz="0.0" izz="4.0"/>
+      </inertial>
       <visual>
         <geometry>
@@ -29,4 +42,7 @@
         </geometry>
         <origin rpy="-0.0 0.0 -0.0" xyz="0.0 0.0 0.0"/>
+        <material name="KukaOrange">
+          <color rgba="1.0 0.4 0.0 1.0"/>
+        </material>
       </visual>
     </link>
@@ -38,4 +54,9 @@
         <origin rpy="-0.0 0.0 -0.0" xyz="0.0 0.0 0.0"/>
       </collision>
+      <inertial>
+        <mass value="5.5E1"/>
+        <origin rpy="0.0 0.0 0.0" xyz="0.49 0.0 0.0"/>
+        <inertia ixx="0.5" ixy="0.0" ixz="0.0" iyy="4.4" iyz="0.0" izz="4.4"/>
+      </inertial>
       <visual>
         <geometry>
@@ -43,4 +64,7 @@
         </geometry>
         <origin rpy="-0.0 0.0 -0.0" xyz="0.0 0.0 0.0"/>
+        <material name="KukaOrange">
+          <color rgba="1.0 0.4 0.0 1.0"/>
+        </material>
       </visual>
     </link>
@@ -52,4 +76,9 @@
         <origin rpy="-0.0 0.0 -0.0" xyz="0.0 0.0 0.0"/>
       </collision>
+      <inertial>
+        <mass value="1.5E1"/>
+        <origin rpy="0.0 0.0 0.0" xyz="0.075 0.0 0.0"/>
+        <inertia ixx="0.3" ixy="0.0" ixz="0.0" iyy="0.5" iyz="0.0" izz="0.5"/>
+      </inertial>
       <visual>
         <geometry>
@@ -57,4 +86,7 @@
         </geometry>
         <origin rpy="-0.0 0.0 -0.0" xyz="0.0 0.0 0.0"/>
+        <material name="KukaOrange">
+          <color rgba="1.0 0.4 0.0 1.0"/>
+        </material>
       </visual>
     </link>
@@ -66,4 +98,9 @@
         <origin rpy="-0.0 0.0 -0.0" xyz="0.0 0.0 0.0"/>
       </collision>
+      <inertial>
+        <mass value="1.2E1"/>
+        <origin rpy="0.0 0.0 0.0" xyz="0.0 0.0 -0.43"/>
+        <inertia ixx="0.74" ixy="0.0" ixz="0.0" iyy="0.74" iyz="0.0" izz="0.05"/>
+      </inertial>
       <visual>
         <geometry>
@@ -71,4 +108,7 @@
         </geometry>
         <origin rpy="-0.0 0.0 -0.0" xyz="0.0 0.0 0.0"/>
+        <material name="KukaOrange">
+          <color rgba="1.0 0.4 0.0 1.0"/>
+        </material>
       </visual>
     </link>
@@ -80,4 +120,9 @@
         <origin rpy="-0.0 0.0 -0.0" xyz="0.0 0.0 0.0"/>
       </collision>
+      <inertial>
+        <mass value="5.0"/>
+        <origin rpy="0.0 0.0 0.0" xyz="0.0 0.0 0.0"/>
+        <inertia ixx="0.03" ixy="0.0" ixz="0.0" iyy="0.03" iyz="0.0" izz="0.03"/>
+      </inertial>
       <visual>
         <geometry>
@@ -85,4 +130,7 @@
         </geometry>
         <origin rpy="-0.0 0.0 -0.0" xyz="0.0 0.0 0.0"/>
+        <material name="KukaOrange">
+          <color rgba="1.0 0.4 0.0 1.0"/>
+        </material>
       </visual>
     </link>
@@ -94,4 +142,9 @@
         <origin rpy="-0.0 0.0 -0.0" xyz="0.0 0.0 0.0"/>
       </collision>
+      <inertial>
+        <mass value="4.0"/>
+        <origin rpy="0.0 0.0 0.0" xyz="0.0 0.0 -0.077"/>
+        <inertia ixx="0.008" ixy="0.0" ixz="0.0" iyy="0.008" iyz="0.0" izz="0.005"/>
+      </inertial>
       <visual>
         <geometry>
@@ -99,4 +152,7 @@
         </geometry>
         <origin rpy="-0.0 0.0 -0.0" xyz="0.0 0.0 0.0"/>
+        <material name="KukaOrange">
+          <color rgba="1.0 0.4 0.0 1.0"/>
+        </material>
       </visual>
     </link>
@@ -107,4 +163,5 @@
       <origin rpy="${-pi} 0.0 -0.0" xyz="0.0 0.0 0.0"/>
       <parent link="${prefix}base_link"/>
+      <dynamics damping="25.0" friction="0.0"/>
     </joint>
     <joint name="${prefix}joint_2" type="revolute">
@@ -114,4 +171,5 @@
       <origin rpy="${pi/2.0} 0.0 -0.0" xyz="0.16 0.0 -0.52"/>
       <parent link="${prefix}link_1"/>
+      <dynamics damping="25.0" friction="0.0"/>
     </joint>
     <joint name="${prefix}joint_3" type="revolute">
@@ -121,4 +179,5 @@
       <origin rpy="0.0 0.0 ${-pi/2.0}" xyz="0.98 0.0 0.0"/>
       <parent link="${prefix}link_2"/>
+      <dynamics damping="5.0" friction="0.0"/>
     </joint>
     <joint name="${prefix}joint_4" type="revolute">
@@ -128,4 +187,5 @@
       <origin rpy="${pi/2.0} 0.0 -0.0" xyz="0.15 0.0 0.0"/>
       <parent link="${prefix}link_3"/>
+      <dynamics damping="1.0" friction="0.0"/>
     </joint>
     <joint name="${prefix}joint_5" type="revolute">
@@ -135,4 +195,5 @@
       <origin rpy="${-pi/2.0} 0.0 -0.0" xyz="0.0 0.0 -0.86"/>
       <parent link="${prefix}link_4"/>
+      <dynamics damping="1.0" friction="0.0"/>
     </joint>
     <joint name="${prefix}joint_6" type="revolute">
@@ -142,4 +203,5 @@
       <origin rpy="${pi/2.0} 0.0 -0.0" xyz="0.0 0.0 0.0"/>
       <parent link="${prefix}link_5"/>
+      <dynamics damping="0.5" friction="0.0"/>
     </joint>
     <!-- ROS-Industrial 'base' frame - equivalent of 'KUKA ROBROOT'-->

Commit message: added ee directly to kuka description

File: src/kuka_robot_descriptions/kuka_cybertech_support/urdf/kr16_r2010_2.urdf (robot description, URDF)
Before this commit: robot kr16_r2010_2, 11 links, 10 joints
Links:
- added link gripper_1, mass 0.24148895332843123; collision mesh filename=package://kuka_cybertech_support/meshes/gripper_ee/collisio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 scale=0.001 0.001 0.001; visual mesh filename=package://kuka_cybertech_support/meshes/gripper_ee/visual/g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 scale=0.001 0.001 0.001
- added link gripper_base_link, mass 0.6392407018829523; collision mesh filename=package://kuka_cybertech_support/meshes/gripper_ee/collisio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 scale=0.001 0.001 0.001; visual mesh filename=package://kuka_cybertech_support/meshes/gripper_ee/visual/b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 scale=0.001 0.001 0.001
- added link gripper_tcp
Joints:
- added joint gripper_mount: type fixed, parent flange, child gripper_base_link, origin xyz=0 0 0 rpy=0 0 0
- added joint gripper_slider: type prismatic, parent gripper_base_link, child gripper_1, origin xyz=0.0 -0.048542 -0.005 rpy=0 0 0, axis 0.0 1.0 0.0, limit lower=0.0 upper=0.09 effort=100 velocity=100
- added joint gripper_tcp_joint: type fixed, parent gripper_base_link, child gripper_tcp, origin xyz=0.0 0.0 0.1 rpy=0 0 0

Commit message: adding scenes for pick_place demo with ee

File: src/kuka_robot_descriptions/kuka_cybertech_support/urdf/kr16_r2010_2.urdf (robot description, URDF)
Before this commit: robot kr16_r2010_2, 14 links, 13 joints
Joints:
- joint gripper_mount: origin xyz=0 0 0 rpy=0 0 0 -> xyz=0 0 0 rpy=0 -1.5707963267948966 0
