Commit message: increased torque in slider ee

File: src/kuka_robot_descriptions/kuka_cybertech_support/urdf/gripper_ee_macro.xacro (robot description, xacro)
@@ -64,5 +64,6 @@
       <child link="${prefix}gripper_1"/>
       <axis xyz="0.0 1.0 0.0"/>
-      <limit upper="0.09" lower="0.0" effort="100" velocity="100"/>
+      <limit upper="0.09" lower="0.0" effort="2000" velocity="0.2"/>
+      <dynamics damping="500.0" friction="200.0"/>
     </joint>
     <link name="${prefix}gripper_tcp"/>

File: src/kuka_robot_descriptions/kuka_cybertech_support/urdf/kr16_r2010_2.urdf (robot description, URDF)
Before this commit: robot kr16_r2010_2, 14 links, 13 joints
Joints:
- joint gripper_slider: limit lower=0.0 upper=0.09 effort=100 velocity=100 -> lower=0.0 upper=0.09 effort=2000 velocity=0.2

Commit message: solving issue with grip

File: src/kuka_robot_descriptions/kuka_cybertech_support/urdf/gripper_ee_macro.xacro (robot description, xacro)
@@ -32,8 +32,16 @@
         <material name="${prefix}gripper_silver"/>
       </visual>
+      <!-- housing block (top of gripper, above the jaws) -->
       <collision>
-        <origin xyz="0 0 0" rpy="0 0 0"/>
+        <origin xyz="0 0 0.0125" rpy="0 0 0"/>
         <geometry>
-          <mesh filename="package://kuka_cybertech_support/meshes/gripper_ee/collision/base_link.stl" scale="0.001 0.001 0.001"/>
+          <box size="0.066 0.099 0.025"/>
+        </geometry>
+      </collision>
+      <!-- fixed jaw (thin wall on +Y side, extending down) -->
+      <collision>
+        <origin xyz="0 0.047 -0.047" rpy="0 0 0"/>
+        <geometry>
+          <box size="0.068 0.006 0.094"/>
         </geometry>
       </collision>
@@ -52,8 +60,9 @@
         <material name="${prefix}gripper_silver"/>
       </visual>
+      <!-- moving jaw modeled as a thin plate so gripping volume is open -->
       <collision>
-        <origin xyz="-0.0 0.048542 0.005" rpy="0 0 0"/>
+        <origin xyz="0 0 -0.0445" rpy="0 0 0"/>
         <geometry>
-          <mesh filename="package://kuka_cybertech_support/meshes/gripper_ee/collision/gripper_1.stl" scale="0.001 0.001 0.001"/>
+          <box size="0.068 0.005 0.089"/>
         </geometry>
       </collision>

File: src/kuka_robot_descriptions/kuka_cybertech_support/urdf/kr16_r2010_2.urdf (robot description, URDF)
Before this commit: robot kr16_r2010_2, 14 links, 13 joints
Links:
- link gripper_1: geometry collision box size=0.068 0.005 0.089; visual mesh filename=package://kuka_cybertech_support/meshes/gripper_ee/visual/g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 scale=0.001 0.001 0.001
- link gripper_base_link: geometry collision box size=0.066 0.099 0.025; collision box size=0.068 0.006 0.094

Commit message: integrated rescaled ee to setup

File: src/kuka_robot_descriptions/kuka_cybertech_support/urdf/gripper_ee_macro.xacro (robot description, xacro)
@@ -21,7 +21,7 @@
     <link name="${prefix}gripper_base_link">
       <inertial>
-        <origin xyz="0.0011702561252768843 0.026454745356582574 -0.013981216174508405" rpy="0 0 0"/>
-        <mass value="0.6392407018829523"/>
-        <inertia ixx="0.001069" iyy="0.000811" izz="0.00063" ixy="5e-06" iyz="0.000241" ixz="-1.1e-05"/>
+        <origin xyz="-0.004489232637892108 -0.018469561788532624 -0.10694364852352554" rpy="0 0 0"/>
+        <mass value="17.259498950839642"/>
+        <inertia ixx="0.259724" iyy="0.197155" izz="0.153142" ixy="0.001156" iyz="0.058493" ixz="-0.00277"/>
       </inertial>
       <visual>
@@ -32,16 +32,16 @@
         <material name="${prefix}gripper_silver"/>
       </visual>
-      <!-- housing block (top of gripper, above the jaws) -->
+      <!-- main body (housing + actuator block, above the jaws) -->
       <collision>
-        <origin xyz="0 0 0.0125" rpy="0 0 0"/>
+        <origin xyz="-0.0065 -0.0965 -0.035" rpy="0 0 0"/>
         <geometry>
-          <box size="0.066 0.099 0.025"/>
+          <box size="0.198 0.297 0.120"/>
         </geometry>
       </collision>
-      <!-- fixed jaw (thin wall on +Y side, extending down) -->
+      <!-- fixed jaw (thin bar on +Y side, extending down) -->
       <collision>
-        <origin xyz="0 0.047 -0.047" rpy="0 0 0"/>
+        <origin xyz="-0.007 0.0445 -0.244" rpy="0 0 0"/>
         <geometry>
-          <box size="0.068 0.006 0.094"/>
+          <box size="0.198 0.015 0.207"/>
         </geometry>
       </collision>
@@ -49,10 +49,10 @@
     <link name="${prefix}gripper_1">
       <inertial>
-        <origin xyz="0.0 4.491218433752553e-07 -0.04450000000000001" rpy="0 0 0"/>
-        <mass value="0.24148895332843123"/>
-        <inertia ixx="0.00016" iyy="0.000252" izz="9.4e-05" ixy="0.0" iyz="0.0" ixz="0.0"/>
+        <origin xyz="-1.0132789659417218e-09 -4.5049275015918155e-07 -0.13350000000000006" rpy="0 0 0"/>
+        <mass value="6.5202017398676455"/>
+        <inertia ixx="0.038861" iyy="0.061347" izz="0.022738" ixy="0.0" iyz="0.0" ixz="0.0"/>
       </inertial>
       <visual>
-        <origin xyz="-0.0 0.048542 0.005" rpy="0 0 0"/>
+        <origin xyz="0.008 0.243458 0.08" rpy="0 0 0"/>
         <geometry>
           <mesh filename="package://kuka_cybertech_support/meshes/gripper_ee/visual/gripper_1.stl" scale="0.001 0.001 0.001"/>
@@ -62,16 +62,16 @@
       <!-- moving jaw modeled as a thin plate so gripping volume is open -->
       <collision>
-        <origin xyz="0 0 -0.0445" rpy="0 0 0"/>
+        <origin xyz="0 0 -0.1335" rpy="0 0 0"/>
         <geometry>
-          <box size="0.068 0.005 0.089"/>
+          <box size="0.204 0.015 0.267"/>
         </geometry>
       </collision>
     </link>
     <joint name="${prefix}gripper_slider" type="prismatic">
-      <origin xyz="0.0 -0.048542 -0.005" rpy="0 0 0"/>
+      <origin xyz="-0.008 -0.243458 -0.08" rpy="0 0 0"/>
       <parent link="${prefix}gripper_base_link"/>
       <child link="${prefix}gripper_1"/>
       <axis xyz="0.0 1.0 0.0"/>
-      <limit upper="0.09" lower="0.0" effort="2000" velocity="0.2"/>
+      <limit upper="0.25" lower="0.0" effort="3000" velocity="0.5"/>
       <dynamics damping="500.0" friction="200.0"/>
     </joint>
@@ -80,5 +80,5 @@
       <parent link="${prefix}gripper_base_link"/>
       <child link="${prefix}gripper_tcp"/>
-      <origin xyz="0.0 0.0 0.1" rpy="0 0 0"/>
+      <origin xyz="0.0 0.0 -0.347" rpy="0 0 0"/>
     </joint>
   </xacro:macro>

File: src/kuka_robot_descriptions/kuka_cybertech_support/urdf/kr16_r2010_2.urdf (robot description, URDF)
Before this commit: robot kr16_r2010_2, 14 links, 13 joints
Links:
- link gripper_1: mass 0.24148895332843123 -> 6.5202017398676455; geometry collision box size=0.204 0.015 0.267; visual mesh filename=package://kuka_cybertech_support/meshes/gripper_ee/visual/g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 scale=0.001 0.001 0.001
- link gripper_base_link: mass 0.6392407018829523 -> 17.259498950839642; geometry collision box size=0.198 0.015 0.207; collision box size=0.198 0.297 0.120
Joints:
- joint gripper_slider: limit lower=0.0 upper=0.09 effort=2000 velocity=0.2 -> lower=0.0 upper=0.25 effort=3000 velocity=0.5; origin xyz=0.0 -0.048542 -0.005 rpy=0 0 0 -> xyz=-0.008 -0.243458 -0.08 rpy=0 0 0
- joint gripper_tcp_joint: origin xyz=0.0 0.0 0.1 rpy=0 0 0 -> xyz=0.0 0.0 -0.347 rpy=0 0 0
